Commit message: Gym

File: poppy_torso_description/urdf/Poppy_Torso.URDF (robot description, URDF)
Before this commit: robot Poppy_Torso, 14 links, 13 joints
Links:
- added link l_hand; collision sphere radius=0.002; visual sphere radius=0.002
- added link r_hand; collision sphere radius=0.002; visual sphere radius=0.002
Joints:
- added joint l_wrist: type fixed, parent l_forearm, child l_hand, origin xyz=0.00 0.21 0.003 rpy=0 0 0
- added joint r_wrist: type fixed, parent r_forearm, child r_hand, origin xyz=0.00 0.21 0.003 rpy=0 0 0
